File: Diagramas de Circuito/BLDC Control/_autosave-BLDC Control.kicad_sch (KiCad schematic)
At the start: 4 parts, among them K1 Relay_SPDT, K2 Relay_SPDT, Q1 Q_NMOS_GDS

Commit message: mais relatorio
Parts:
- added J1: BATT_CONN, symbol Connector:Conn_01x02_Pin
- added J2: RASPI_CONN, symbol Connector:Conn_01x03_Socket
- added J3: RASPI_CONN2, symbol Connector:Conn_01x01_Socket
- added U1: ~, symbol SKID_BLDC:CONTROLLER
Connections:
- net GND: now also J2.1 (Pin_1), U1. (SIG)
- net at K1.11: now also U1. (SIG)
- net at Q1.1 (G): now also J3.1 (Pin_1)
- net at M1.2: now also U1. (SIG)
- net at K2.11: now also U1. (SIG)
- new net: J2.2 (Pin_2), U1. (SIG)
- new net: J2.3 (Pin_3), U1. (SIG)
- new net: J1.1 (Pin_1), U1. (SIG)
- new net: J1.2 (Pin_2), U1. (SIG)
